Commit message: Added depth camera

File: turtlebot3_gazebo/urdf/turtlebot3_waffle_pi.urdf (robot description, URDF)
Before this commit: robot turtlebot3_waffle_pi, 11 links, 10 joints
Links:
- added link camera_depth_link
- added link camera_depth_optical_frame
Joints:
- added joint camera_depth_joint: type fixed, parent camera_link, child camera_depth_link, origin xyz=0.003 0.011 0.009 rpy=-1.57 0 -1.57
- added joint camera_depth_optical_joint: type fixed, parent camera_depth_link, child camera_depth_optical_frame, origin xyz=0 0 0 rpy=-1.57 0 -1.57
